File: schematics/HARE - Master Schematic v1.0.sch (EAGLE design)
At the start: 96 parts, among them IC1 NE5532N, IC2 NE5532N, IC3 FT232RL, IC4 NE5532N, IC5 7805DT, IC6 AT25P, J1 9V, J2 STEREOSW, J3 STEREOSW, Q1 16 MHz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

Commit message: Updated the board file to include cutout for foot switch and some greenburg recommendations
Parts:
- removed SW1: 3PDT, gm-switches:3PDT
- added SV1: FtSW1, con-lstb:MA03-1
- added SV2: FtSW2, con-lstb:MA03-1
Connections:
- removed net BYPASS: SW1A.3, SW1C.3
- removed net N$15: APOT1.2, SW1C.1
- removed net N$19: J3.T, J3.TN, SW1C.2
- removed net N$9: C1.1, SW1A.1
- new net A_IN: C1.1, SV1.2
- new net A_OUT: APOT1.2, SV2.3
- new net OUTPUT: J3.T, J3.TN, SV2.2
- new net PWR_LED: D1.C, SV1.3
- net DAC_CS: now also R29.1, U2.~CS; no longer IC6.HOLD/, R7.2
- net GND: now also SV2.1; no longer SW1B.2
- net INPUT: now also SV1.1; no longer SW1A.2, SW1B.3
- net MEM_CS: no longer R29.1, U2.~CS
- net N$8: now also IC6.HOLD/, R7.2; no longer D1.C, SW1B.1
Other:
- note added: "Foot Switch Connector"
Changed lines of the file:
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@@
 <part name="APOT1" library="gm-pots" deviceset="POT" device="S" value="100k"/>
 <part name="APOT2" library="gm-pots" deviceset="POT" device="S" value="250k"/>
-<part name="SW1" library="gm-switches" deviceset="3PDT" device="" value="3PDT"/>
 <part name="IC3" library="ftdichip" library_urn="urn:adsk.eagle:library:231" deviceset="FT232R" device="L" package3d_urn="urn:adsk.eagle:package:14013/1"/>
 <part name="X2" library="con-usb" deviceset="USB" device="-B-H"/>
@@
 <part name="R29" library="resistor" library_urn="urn:adsk.eagle:library:348" deviceset="R-US_" device="R0805" package3d_urn="urn:adsk.eagle:package:26059/1" value="10k"/>
 <part name="C29" library="resistor" library_urn="urn:adsk.eagle:library:348" deviceset="C-EU" device="C0805K" package3d_urn="urn:adsk.eagle:package:26201/1" value="1uF"/>
+<part name="SV2" library="con-lstb" library_urn="urn:adsk.eagle:library:162" deviceset="MA03-1" device="" package3d_urn="urn:adsk.eagle:package:8339/1" value="FtSW2"/>
+<part name="SUPPLY43" library="supply2" library_urn="urn:adsk.eagle:library:372" deviceset="GND" device=""/>
+<part name="SV1" library="con-lstb" library_urn="urn:adsk.eagle:library:162" deviceset="MA03-1" device="" package3d_urn="urn:adsk.eagle:package:8339/1" value="FtSW1"/>
 </parts>
 <sheets>
@@
 <text x="462.28" y="33.02" size="3.81" layer="97" ratio="14">The H.A.R.E Project - ECE411</text>
 <text x="551.18" y="12.7" size="3.81" layer="97" font="vector" ratio="15">D</text>
+<text x="365.76" y="167.64" size="3.81" layer="97" font="vector" ratio="12">Foot Switch Connector</text>
 </plain>
 <instances>
@@
 <instance part="APOT1" gate="G$1" x="281.94" y="119.38" rot="MR180"/>
 <instance part="APOT2" gate="G$1" x="266.7" y="106.68"/>
-<instance part="SW1" gate="A" x="58.42" y="218.44" rot="R270"/>
-<instance part="SW1" gate="B" x="464.82" y="350.52" rot="R270"/>
-<instance part="SW1" gate="C" x="299.72" y="116.84" rot="MR270"/>
 <instance part="IC3" gate="1" x="210.82" y="340.36"/>
 <instance part="X2" gate="G$1" x="162.56" y="322.58" rot="MR0"/>
@@
 <instance part="R29" gate="G$1" x="195.58" y="236.22" rot="R90"/>
 <instance part="C29" gate="G$1" x="124.46" y="238.76" rot="R180"/>
+<instance part="SV2" gate="G$1" x="381" y="147.32"/>
+<instance part="SUPPLY43" gate="GND" x="408.94" y="137.16"/>
+<instance part="SV1" gate="G$1" x="383.54" y="111.76"/>
 </instances>
 <busses>
@@
 </segment>
 <segment>
-<pinref part="SW1" gate="B" pin="2"/>
 <wire x1="459.74" y1="350.52" x2="454.66" y2="350.52" width="0.1524" layer="91"/>
 <pinref part="SUPPLY4" gate="GND" pin="GND"/>
@@
 <wire x1="124.46" y1="236.22" x2="124.46" y2="231.14" width="0.1524" layer="91"/>
 </segment>
+<segment>
+<pinref part="SV2" gate="G$1" pin="1"/>
+<wire x1="388.62" y1="144.78" x2="398.78" y2="144.78" width="0.1524" layer="91"/>
+<wire x1="398.78" y1="144.78" x2="398.78" y2="139.7" width="0.1524" layer="91"/>
+<wire x1="398.78" y1="139.7" x2="408.94" y2="139.7" width="0.1524" layer="91"/>
+<pinref part="SUPPLY43" gate="GND" pin="GND"/>
+</segment>
 </net>
 <net name="INPUT" class="0">
 <segment>
 <wire x1="40.64" y1="236.22" x2="45.72" y2="236.22" width="0.1524" layer="91"/>
-<pinref part="SW1" gate="A" pin="2"/>
 <wire x1="45.72" y1="236.22" x2="45.72" y2="233.68" width="0.1524" layer="91"/>
 <wire x1="45.72" y1="233.68" x2="45.72" y2="218.44" width="0.1524" layer="91"/>
@@
 </segment>
 <segment>
-<pinref part="SW1" gate="B" pin="3"/>
 <wire x1="469.9" y1="347.98" x2="477.52" y2="347.98" width="0.1524" layer="91"/>
 <label x="477.52" y="347.98" size="1.27" layer="95" font="vector" ratio="12" xref="yes"/>
+<label x="408.94" y="109.22" size="1.27" layer="95" font="vector" ratio="12" xref="yes"/>
+</segment>
+<segment>
+<wire x1="388.62" y1="109.22" x2="391.16" y2="109.22" width="0.1524" layer="91"/>
+<pinref part="SV1" gate="G$1" pin="1"/>
+<wire x1="391.16" y1="109.22" x2="408.94" y2="109.22" width="0.1524" layer="91"/>
+<junction x="391.16" y="109.22"/>
 </segment>
 </net>
@@
 </segment>
 </net>
-<net name="N$8" class="0">
+<net name="PWR_LED" class="0">
 <segment>
 <pinref part="D1" gate="G$1" pin="C"/>
 <wire x1="472.44" y1="358.14" x2="472.44" y2="353.06" width="0.1524" layer="91"/>
-<pinref part="SW1" gate="B" pin="1"/>
 <wire x1="472.44" y1="353.06" x2="469.9" y2="353.06" width="0.1524" layer="91"/>
-</segment>
-</net>
-<net name="N$9" class="0">
-<segment>
-<pinref part="SW1" gate="A" pin="1"/>
+<label x="469.9" y="353.06" size="1.778" layer="95"/>
+</segment>
+<segment>
+<wire x1="388.62" y1="114.3" x2="391.16" y2="114.3" width="0.1524" layer="91"/>
+<wire x1="391.16" y1="114.3" x2="408.94" y2="114.3" width="0.1524" layer="91"/>
+<pinref part="SV1" gate="G$1" pin="3"/>
+<junction x="391.16" y="114.3"/>
+<label x="408.94" y="114.3" size="1.778" layer="95"/>
+</segment>
+</net>
+<net name="A_IN" class="0">
+<segment>
 <wire x1="63.5" y1="220.98" x2="71.12" y2="220.98" width="0.1524" layer="91"/>
 <wire x1="71.12" y1="220.98" x2="71.12" y2="236.22" width="0.1524" layer="91"/>
 <pinref part="C1" gate="G$1" pin="1"/>
 <wire x1="71.12" y1="236.22" x2="73.66" y2="236.22" width="0.1524" layer="91"/>
+<label x="63.5" y="220.98" size="1.778" layer="95"/>
+</segment>
+<segment>
+<wire x1="388.62" y1="111.76" x2="391.16" y2="111.76" width="0.1524" layer="91"/>
+<wire x1="391.16" y1="111.76" x2="408.94" y2="111.76" width="0.1524" layer="91"/>
+<pinref part="SV1" gate="G$1" pin="2"/>
+<junction x="391.16" y="111.76"/>
+<label x="408.94" y="111.76" size="1.778" layer="95"/>
 </segment>
 </net>
@@
 <net name="BYPASS" class="0">
 <segment>
-<pinref part="SW1" gate="A" pin="3"/>
 <wire x1="63.5" y1="215.9" x2="73.66" y2="215.9" width="0.1524" layer="91"/>
 <wire x1="73.66" y1="215.9" x2="73.66" y2="210.82" width="0.1524" layer="91"/>
 <label x="73.66" y="210.82" size="1.6764" layer="95" rot="R270" xref="yes"/>
+<label x="63.5" y="215.9" size="1.6764" layer="95" rot="R270" xref="yes"/>
 </segment>
 <segment>
 <wire x1="294.64" y1="114.3" x2="294.64" y2="106.68" width="0.1524" layer="91"/>
 <label x="294.64" y="106.68" size="1.6764" layer="95" rot="R270" xref="yes"/>
-<pinref part="SW1" gate="C" pin="3"/>
-</segment>
-</net>
-<net name="N$19" class="0">
+<label x="294.64" y="114.3" size="1.6764" layer="95" xref="yes"/>
+</segment>
+</net>
+<net name="OUTPUT" class="0">
 <segment>
 <wire x1="304.8" y1="116.84" x2="304.8" y2="144.78" width="0.1524" layer="91"/>
@@
 <wire x1="304.8" y1="147.32" x2="304.8" y2="144.78" width="0.1524" layer="91"/>
 <junction x="304.8" y="144.78"/>
-<pinref part="SW1" gate="C" pin="2"/>
+<label x="304.8" y="116.84" size="1.778" layer="95" rot="R90"/>
+</segment>
+<segment>
+<pinref part="SV2" gate="G$1" pin="2"/>
+<wire x1="388.62" y1="147.32" x2="408.94" y2="147.32" width="0.1524" layer="91"/>
+<label x="408.94" y="147.32" size="1.778" layer="95"/>
 </segment>
 </net>
@@
 </segment>
 </net>
-<net name="N$15" class="0">
+<net name="A_OUT" class="0">
 <segment>
 <pinref part="APOT1" gate="G$1" pin="2"/>
-<pinref part="SW1" gate="C" pin="1"/>
 <wire x1="284.48" y1="119.38" x2="294.64" y2="119.38" width="0.1524" layer="91"/>
+<label x="292.1" y="119.38" size="1.778" layer="95"/>
+</segment>
+<segment>
+<pinref part="SV2" gate="G$1" pin="3"/>
+<wire x1="388.62" y1="149.86" x2="398.78" y2="149.86" width="0.1524" layer="91"/>
+<wire x1="398.78" y1="149.86" x2="398.78" y2="154.94" width="0.1524" layer="91"/>
+<wire x1="398.78" y1="154.94" x2="408.94" y2="154.94" width="0.1524" layer="91"/>
+<label x="408.94" y="154.94" size="1.778" layer="95"/>
 </segment>
 </net>
@@
 </segment>
 <segment>
-<pinref part="IC6" gate="G$1" pin="HOLD/"/>
-<wire x1="314.96" y1="365.76" x2="320.04" y2="365.76" width="0.1524" layer="91"/>
-<wire x1="320.04" y1="365.76" x2="320.04" y2="381" width="0.1524" layer="91"/>
-<pinref part="R7" gate="G$1" pin="2"/>
+<pinref part="U2" gate="A" pin="~CS"/>
+<wire x1="210.82" y1="228.6" x2="195.58" y2="228.6" width="0.1524" layer="91"/>
+<label x="193.04" y="228.6" size="1.016" layer="95" rot="R180" xref="yes"/>
+<wire x1="195.58" y1="228.6" x2="193.04" y2="228.6" width="0.1524" layer="91"/>
+<wire x1="195.58" y1="228.6" x2="195.58" y2="231.14" width="0.1524" layer="91"/>
+<junction x="195.58" y="228.6"/>
+<pinref part="R29" gate="G$1" pin="1"/>
 </segment>
 </net>
@@
 <net name="MEM_CS" class="0">
 <segment>
-<pinref part="U2" gate="A" pin="~CS"/>
-<wire x1="210.82" y1="228.6" x2="195.58" y2="228.6" width="0.1524" layer="91"/>
-<label x="193.04" y="228.6" size="1.016" layer="95" rot="R180" xref="yes"/>
-<wire x1="195.58" y1="228.6" x2="193.04" y2="228.6" width="0.1524" layer="91"/>
-<wire x1="195.58" y1="228.6" x2="195.58" y2="231.14" width="0.1524" layer="91"/>
-<junction x="195.58" y="228.6"/>
-<pinref part="R29" gate="G$1" pin="1"/>
-</segment>
-<segment>
 <wire x1="114.3" y1="345.44" x2="119.38" y2="345.44" width="0.1524" layer="91"/>
 <label x="119.38" y="345.44" size="1.016" layer="95" xref="yes"/>
@@
 </segment>
 </net>
+<net name="N$8" class="0">
+<segment>
+<pinref part="IC6" gate="G$1" pin="HOLD/"/>
+<wire x1="314.96" y1="365.76" x2="320.04" y2="365.76" width="0.1524" layer="91"/>
+<pinref part="R7" gate="G$1" pin="2"/>
+<wire x1="320.04" y1="365.76" x2="320.04" y2="381" width="0.1524" layer="91"/>
+</segment>
+</net>
