File: schematics/HARE - 3PDT Breakout Schematic v1.0.sch (EAGLE design)
At the start: 4 parts, among them SW1 3PDTBLUE

Commit message: adapting 3PDT breakout board to mate with HARE main board
Parts:
- removed SV3: (no value), con-lstb:MA03-1
Connections:
- net ANALOG_IN: now also SV1.2; no longer SV1.1
- net ANALOG_OUT: now also SV2.3; no longer SV3.2
- net BYPASS: no longer SV1.3, SV3.3
- net GND: now also SV2.1; no longer SV2.2
- net INPUT: now also SV1.1; no longer SV1.2, SV2.3
- net OUTPUT: now also SV2.2; no longer SV3.1
- net PWR_LED: now also SV1.3; no longer SV2.1
Changed lines of the file:
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@@
 <?xml version="1.0" encoding="utf-8"?>
 <!DOCTYPE eagle SYSTEM "eagle.dtd">
-<eagle version="8.4.0">
+<eagle version="8.4.1">
 <drawing>
 <settings>
@@
 <part name="SV1" library="con-lstb" deviceset="MA03-1" device=""/>
 <part name="SV2" library="con-lstb" deviceset="MA03-1" device=""/>
-<part name="SV3" library="con-lstb" deviceset="MA03-1" device=""/>
 </parts>
 <sheets>
@@
 <instance part="SV1" gate="G$1" x="55.88" y="93.98" rot="R180"/>
 <instance part="SV2" gate="G$1" x="132.08" y="93.98" rot="R180"/>
-<instance part="SV3" gate="G$1" x="213.36" y="93.98" rot="R180"/>
 </instances>
 <busses>
@@
 </segment>
 <segment>
-<pinref part="SV1" gate="G$1" pin="2"/>
-<wire x1="48.26" y1="93.98" x2="43.18" y2="93.98" width="0.1524" layer="91"/>
-<label x="43.18" y="93.98" size="1.016" layer="95" rot="R180" xref="yes"/>
-</segment>
-<segment>
-<label x="119.38" y="91.44" size="1.016" layer="95" rot="R180" xref="yes"/>
-<pinref part="SV2" gate="G$1" pin="3"/>
-<wire x1="124.46" y1="91.44" x2="119.38" y2="91.44" width="0.1524" layer="91"/>
+<wire x1="48.26" y1="96.52" x2="40.64" y2="96.52" width="0.1524" layer="91"/>
+<label x="40.64" y="96.52" size="1.016" layer="95" rot="R180" xref="yes"/>
+<pinref part="SV1" gate="G$1" pin="1"/>
+<junction x="48.26" y="96.52"/>
 </segment>
 </net>
@@
 </segment>
 <segment>
-<pinref part="SV1" gate="G$1" pin="1"/>
-<wire x1="48.26" y1="96.52" x2="43.18" y2="96.52" width="0.1524" layer="91"/>
-<label x="43.18" y="96.52" size="1.016" layer="95" rot="R180" xref="yes"/>
+<wire x1="48.26" y1="93.98" x2="40.64" y2="93.98" width="0.1524" layer="91"/>
+<label x="40.64" y="93.98" size="1.016" layer="95" rot="R180" xref="yes"/>
+<pinref part="SV1" gate="G$1" pin="2"/>
+<junction x="48.26" y="93.98"/>
 </segment>
 </net>
@@
 <label x="226.06" y="96.52" size="2.54" layer="95" rot="R270" xref="yes"/>
 </segment>
-<segment>
-<pinref part="SV1" gate="G$1" pin="3"/>
-<wire x1="48.26" y1="91.44" x2="43.18" y2="91.44" width="0.1524" layer="91"/>
-<label x="43.18" y="91.44" size="1.016" layer="95" rot="R180" xref="yes"/>
-</segment>
-<segment>
-<wire x1="205.74" y1="91.44" x2="200.66" y2="91.44" width="0.1524" layer="91"/>
-<label x="200.66" y="91.44" size="1.016" layer="95" rot="R180" xref="yes"/>
-<pinref part="SV3" gate="G$1" pin="3"/>
-</segment>
 </net>
 <net name="ANALOG_OUT" class="0">
@@
 </segment>
 <segment>
-<wire x1="205.74" y1="93.98" x2="200.66" y2="93.98" width="0.1524" layer="91"/>
-<label x="200.66" y="93.98" size="1.016" layer="95" rot="R180" xref="yes"/>
-<pinref part="SV3" gate="G$1" pin="2"/>
+<wire x1="124.46" y1="91.44" x2="116.84" y2="91.44" width="0.1524" layer="91"/>
+<label x="116.84" y="91.44" size="1.016" layer="95" rot="R180" xref="yes"/>
+<pinref part="SV2" gate="G$1" pin="3"/>
+<junction x="124.46" y="91.44"/>
 </segment>
 </net>
@@
 </segment>
 <segment>
-<label x="119.38" y="96.52" size="1.016" layer="95" rot="R180" xref="yes"/>
-<pinref part="SV2" gate="G$1" pin="1"/>
-<wire x1="119.38" y1="96.52" x2="124.46" y2="96.52" width="0.1524" layer="91"/>
+<label x="40.64" y="91.44" size="1.016" layer="95" rot="R180" xref="yes"/>
+<wire x1="40.64" y1="91.44" x2="48.26" y2="91.44" width="0.1524" layer="91"/>
+<pinref part="SV1" gate="G$1" pin="3"/>
+<junction x="48.26" y="91.44"/>
 </segment>
 </net>
@@
 </segment>
 <segment>
-<wire x1="205.74" y1="96.52" x2="200.66" y2="96.52" width="0.1524" layer="91"/>
-<label x="200.66" y="96.52" size="1.016" layer="95" rot="R180" xref="yes"/>
-<pinref part="SV3" gate="G$1" pin="1"/>
+<wire x1="124.46" y1="93.98" x2="116.84" y2="93.98" width="0.1524" layer="91"/>
+<label x="116.84" y="93.98" size="1.016" layer="95" rot="R180" xref="yes"/>
+<pinref part="SV2" gate="G$1" pin="2"/>
+<junction x="124.46" y="93.98"/>
 </segment>
 </net>
@@
 </segment>
 <segment>
-<wire x1="124.46" y1="93.98" x2="119.38" y2="93.98" width="0.1524" layer="91"/>
-<label x="119.38" y="93.98" size="1.016" layer="95" rot="R180" xref="yes"/>
-<pinref part="SV2" gate="G$1" pin="2"/>
-</segment>
-</net>
+<wire x1="124.46" y1="96.52" x2="116.84" y2="96.52" width="0.1524" layer="91"/>
+<label x="116.84" y="96.52" size="1.016" layer="95" rot="R180" xref="yes"/>
+<pinref part="SV2" gate="G$1" pin="1"/>
+<junction x="124.46" y="96.52"/>
+</segment>
+</net>

Commit message: Correctly placed the 3PDT switch connectors to mate with the main board
Parts:
- SV1: value (none) -> FtSW1
- SV2: value (none) -> FtSW2
Changed lines of the file:
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@@
 <parts>
 <part name="SW1" library="gm-switches" deviceset="3PDT" device="BLUE"/>
-<part name="FRAME1" library="frames" deviceset="FRAME_A_L" device=""/>
-<part name="SV1" library="con-lstb" deviceset="MA03-1" device=""/>
-<part name="SV2" library="con-lstb" deviceset="MA03-1" device=""/>
+<part name="FRAME1" library="frames" deviceset="FRAME_A_L" device="" value="3PDT Breakout Board"/>
+<part name="SV1" library="con-lstb" deviceset="MA03-1" device="" value="FtSW1"/>
+<part name="SV2" library="con-lstb" deviceset="MA03-1" device="" value="FtSW2"/>
 </parts>
 <sheets>
